File: Hardware/Logomatic.sch (EAGLE design)
At the start: 63 parts, among them Q1 12MHz, Q2 32kHz, Q4 TRANSISTOR_PNPSMD, U1 MCP73831, U2 3.3V, U3 USD-SOCKETNEW, U4 LPC213X, X1 USBSMD

Commit message: Version 2.7 board commit
Parts:
- removed U$9: CREATIVE_COMMONS, SparkFun:CREATIVE_COMMONS
- added FRAME2, FRAME4: FRAME-LETTER, SparkFun-Aesthetics:FRAME-LETTER
- added LOGO1: OSHW-LOGOL, SparkFun-Aesthetics:OSHW-LOGOL
- added LOGO2: SFE_LOGO_NAME.1_INCH, SparkFun-Aesthetics:SFE_LOGO_NAME.1_INCH
- added U$10: REVISION, SparkFun-Aesthetics:REVISION
- C1, C10, C11, C12, C2, C7, C8, C9: device SparkFunEagle-6-6-07:CAP0402 -> SparkFun-Capacitors:0.1UF-25V(+80/-20%)(0603)
- C13, C14, C15, C16: device SparkFunEagle-6-6-07:CAP0402 -> SparkFun-Capacitors:22PF-50V-5%(0603)
- C17, C5: device SparkFun:CAP0402-CAP -> SparkFun-Capacitors:4.7UF-6.3V-10%(0603)0603
- C3, C4: device SparkFunEagle-6-6-07:CAP0402 -> SparkFun-Capacitors:18PF-50V-5%(0603)
- C6: device SparkFun:CAP_POL1206 -> SparkFun-Capacitors:10UF-16V-10%(TANT)
- R1, R13, R6, R7, R8: device SparkFunEagle-6-6-07:RESISTOR0402 -> SparkFun-Resistors:10KOHM1/10W1%(0603)0603
- R10, R9: device SparkFunEagle-6-6-07:RESISTOR0402 -> SparkFun-Resistors:33OHM1/10W1%(0603)
- R11: device SparkFunEagle-6-6-07:RESISTOR0402 -> SparkFun-Resistors:1.5KOHM1/10W1%(0603)
- R12: device SparkFunEagle-6-6-07:RESISTOR0402 -> SparkFun-Resistors:1KOHM1/10W1%(0603)
- R14: device SparkFunEagle-6-6-07:RESISTOR0402 -> SparkFun-Resistors:100KOHM1/10W1%(0603)
- R15, R4, R5: device SparkFunEagle-6-6-07:RESISTOR0402 -> SparkFun-Resistors:330OHM1/10W1%(0603)
- R16, R17: device SparkFun:RESISTOR0402-RES -> SparkFun-Resistors:1MOHM1/10W1%(0603)
- R2: device SparkFun:RESISTOR0402-RES -> SparkFun-Resistors:2.0KOHM1/10W5%(0603)
- R3: device SparkFun:RESISTOR0402-RES -> SparkFun-Resistors:330OHM1/10W1%(0603)
- U$6: value LOGO-SFENEW -> SFE_LOGO_FLAME1_INCH; device SparkFun:LOGO-SFENEW -> SparkFun-Aesthetics:SFE_LOGO_FLAME1_INCH
- U3: device SparkFun:USD-SOCKETNEW -> SparkFun-Connectors:USD-SOCKETNEW
- X1: value USBSMD -> USB_MICROB_PLUGCONN-11752; device SparkFun:USBSMD -> SparkFun-Connectors:USB_MICROB_PLUGCONN-11752
Connections:
- net USB_VIN: now also X1.VCC; no longer X1.VBUS
Other:
- note added: "Toni Klopfenstein"
- note added: "v2.7"

Commit message: Updating to fancy new silk on board
Parts:
- added LOGO3: SFE_LOGO_FLAME.4_INCH, SparkFun-Aesthetics:SFE_LOGO_FLAME.4_INCH
- U$6: value SFE_LOGO_FLAME1_INCH -> LOGOMATIC_LOGO; device SparkFun-Aesthetics:SFE_LOGO_FLAME1_INCH -> SparkFun-Aesthetics:LOGOMATIC_LOGO
Changed lines of the file:
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@@
 <part name="P+14" library="SparkFunEagle-6-6-07" deviceset="VCC" device=""/>
 <part name="C11" library="SparkFun-Capacitors" deviceset="0.1UF-25V(+80/-20%)(0603)" device="" value="0.1uF"/>
-<part name="U$6" library="SparkFun-Aesthetics" deviceset="SFE_LOGO_FLAME" device="1_INCH"/>
 <part name="FRAME4" library="SparkFun-Aesthetics" deviceset="FRAME-LETTER" device=""/>
 <part name="C6" library="SparkFun-Capacitors" deviceset="10UF-16V-10%(TANT)" device="" value="10uF"/>
@@
 <part name="LOGO1" library="SparkFun-Aesthetics" deviceset="OSHW-LOGO" device="L"/>
 <part name="LOGO2" library="SparkFun-Aesthetics" deviceset="SFE_LOGO_NAME" device=".1_INCH"/>
+<part name="U$6" library="SparkFun-Aesthetics" deviceset="LOGOMATIC_LOGO" device=""/>
+<part name="LOGO3" library="SparkFun-Aesthetics" deviceset="SFE_LOGO_FLAME" device=".4_INCH" value="SFE_LOGO_FLAME.4_INCH"/>
 </parts>
 <sheets>
@@
 <instance part="P+14" gate="1" x="162.56" y="134.62"/>
 <instance part="C11" gate="G$1" x="162.56" y="127"/>
-<instance part="U$6" gate="G$1" x="238.76" y="35.56"/>
 <instance part="U$10" gate="G$1" x="149.098" y="7.112"/>
 <instance part="LOGO1" gate="G$1" x="134.62" y="10.16"/>
 <instance part="LOGO2" gate="G$1" x="180.34" y="33.02"/>
+<instance part="U$6" gate="G$1" x="91.44" y="0"/>
+<instance part="LOGO3" gate="G$1" x="238.76" y="35.56"/>
 </instances>
 <busses>

Commit message: Changing 0603 LED package
Parts:
- LED1: device SparkFun:LED0603 -> SparkFun-LED:LED-RED0603
- LED2: device SparkFunEagle-6-6-07:LED0603 -> SparkFun-LED:LED-RED0603
- LED3: device SparkFun_Master:LED0603 -> SparkFun-LED:LED-RED0603
- LED4: device SparkFunEagle-6-6-07:LED0603 -> SparkFun-LED:LED-GREEN0603
Changed lines of the file:
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@@
 <part name="GND14" library="SparkFun" deviceset="GND" device=""/>
 <part name="GND15" library="SparkFun" deviceset="GND" device=""/>
-<part name="LED3" library="SparkFun_Master" deviceset="LED" device="0603"/>
+<part name="LED3" library="SparkFun-LED" deviceset="LED-RED" device="0603"/>
 <part name="FRAME2" library="SparkFun-Aesthetics" deviceset="FRAME-LETTER" device=""/>
 <part name="X1" library="SparkFun-Connectors" deviceset="USB_MICROB_PLUG" device="CONN-11752"/>
@@
 <part name="P+12" library="SparkFunEagle-6-6-07" deviceset="VCC" device=""/>
 <part name="S3" library="SparkFunEagle-6-6-07" deviceset="TAC_SWITCH" device="SND" value="Reset"/>
-<part name="LED2" library="SparkFunEagle-6-6-07" deviceset="LED" device="0603" value="RED"/>
-<part name="LED4" library="SparkFunEagle-6-6-07" deviceset="LED" device="0603" value="GREEN"/>
+<part name="LED2" library="SparkFun-LED" deviceset="LED-RED" device="0603" value="RED"/>
+<part name="LED4" library="SparkFun-LED" deviceset="LED-GREEN" device="0603" value="GREEN"/>
 <part name="Q1" library="SparkFunEagle-6-6-07" deviceset="CRYSTAL" device="5X3" value="12MHz"/>
 <part name="GND18" library="SparkFunEagle-6-6-07" deviceset="GND" device=""/>
@@
 <part name="GND16" library="SparkFun" deviceset="GND" device=""/>
 <part name="GND20" library="SparkFun" deviceset="GND" device=""/>
-<part name="LED1" library="SparkFun" deviceset="LED" device="0603" value="LED RED"/>
+<part name="LED1" library="SparkFun-LED" deviceset="LED-RED" device="0603" value="LED RED"/>
 <part name="JP2" library="SparkFun" deviceset="M02" device="-JST-2MM-SMT" value="LiPo"/>
 <part name="JP5" library="SparkFun" deviceset="M06" device="SIP"/>

Commit message: Sorted gitignore
Parts:
- removed U3: USD-SOCKETNEW, SparkFun-Connectors:USD-SOCKETNEW
- added J1: USD_CONNECTOR, SparkFun-Connectors:USD_CONNECTOR
- added R18, R19, R20: 100k, SparkFun-Resistors:100KOHM-1/10W-1%(0603)
- R2: value 2K -> 2.0k
Connections:
- removed net CS0: U3.CS, U4.(SSEL0/PWM2/EINT2)P0.7
- new net !CS0: J1.!CS, U4.(SSEL0/PWM2/EINT2)P0.7
- new net CD: J1.CD2
- new net N$10: J1.RSV@2, R19.1
- new net N$3: J1.CD1, R18.1
- new net N$4: J1.RSV@1, R20.1
- net GND: now also J1.GND, J1.SHIELD@1, J1.SHIELD@3; no longer U3.GND, U3.SHIELD@3, U3.SHIELD@4
- net MISO0: now also J1.DO; no longer U3.DO
- net MOSI0: now also J1.DI; no longer U3.DI
- net SCK0: now also J1.SCK; no longer U3.SCK
- net VCC: now also J1.VCC, R18.2, R19.2, R20.2; no longer U3.VCC
